File: hardware/io-board/controlboard.kicad_sch (KiCad schematic)
At the start: 45 parts

Commit message: Recover from the backup notes on the schematic (errata, etc.)
Connections:
- no-connect marks 8 -> 9
Other:
- note added: "- CAN / RS485 cables on board suggest pair-by-pair setting - not T-568B. This will distinguish cables too. But both approaches can work. - Suggested layout: Full-color for ground (on IO_CAN), Pair order: orange, green, blue, brown. IO-CAN Socket and RJ45 connector therefore: w-o o, w-g g, w-bl bl, w-br br (1 2, 3 4, 5 6, 7 8). That keeps CAN as orange pair, forwarded as brown pair. Main power on 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"
- note added: "BOOT0!"
- note added: "Board v1 errors, to be corrected: - EVDS footprint doesn't match my device. - Battery is smaller and can be shifted right. - Can CAP can be outside. - some labels can be moved a bit away for eligibility - CAPs don't have GND marked. - Mark ground on power pins - holes of CPU could be larger - HI_STAB footprint could use double pinheader. Single is wobbly (and impossible to buy, one has to cut it)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"
- note added: "Board v1 ideas, maybe? - Add a pin in another axis in i2c connector for stabilization. Say - duplicated GND/VCC."
- note added: "CAN uses PB8 that is also BOOT0. You need to select nBOOT_SEL to free the GPIO, otherwise the board won't boot."
- note added: "PCF8575 expander "modules": - Might have 3.3V stabilizer onboard which is not required; PCF can handle 6.5V absolute. - Have pull-ups for SDA/SCL for VCC which is NOT required and problematic. - Can handle VCC+0.5V input voltage max so 3.8V with stab. - Can't safely drive 5V "low level trigger" devices. I suggest shorting the onboard 3.3V stab to get 5V PCF and removing/shorting the sda/scl pull-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"
- note removed: "- CAN / RS485 cables on board suggest pair-by-pair setting. Not T-568B - Board could be powered by USB (weact board has a vbus->vcc diode). Also connecting USB while board is powered externally should not break anything. - Keep empty space over the screws to allow for a HAT or another layer. 50x100 fits the SSR relay board too. - CAN Forwarding jumpers allow to construct a linear bus in situation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"
